File: hw/subbat.kicad_pcb (KiCad board)
At the start: 2 copper layers, 100 x 100 mm, 154 parts, among them J1 Conn_01x02, J10 Conn_01x06_Male, J11 USB_Ax2, J12 USB_Ax2, J13 USB_Ax2, J14 Conn_01x05_Female, J15 Conn_01x04_Male, J16 Conn_01x06_Male, J17 Conn_01x06_Male, J2 Conn_01x02, J3 Conn_01x02, J4 Conn_01x02, J5 Conn_01x02, J6 Conn_01x02, J7 Conn_01x06_Male, J8 Conn_01x02, J9 USB_Ax2, Q1 Q_NPN_BEC, Q10 Q_NPN_BEC, Q11 AOD403, Q12 AOD403, Q13 Q_NPN_BEC, Q14 AOD403, Q15 Q_NPN_BEC, Q16 Q_NPN_BEC, Q17 Q_PMOS_GSD, Q2 Q_PMOS_GSD, Q3 AOD403, Q4 Q_NPN_BEC, Q5 AOD403, Q6 AOD403, Q7 Q_NPN_BEC, Q8 AOD403, Q9 AOD403, SW1 SW_Push, SW2 SW_Push, SW3 SW_Push, U1 ATMEGA328P-PU, U2 L7805, U3 ATTINY2313-20PU, U4 ATTINY13A-PU, U5 LT6105, U6 LT6105

Commit message: Added current sensors; and other many modifications
Parts:
- added C22: 1u, Capacitors_SMD:C_0603_HandSoldering, F.Cu at (33.0, 38.5)
- added C23: 1u, Capacitors_SMD:C_0603_HandSoldering, B.Cu at (106.8, 97.8)
- added R45: 0.01R, Resistors_SMD:R_2512, B.Cu at (30.5, 35.0)
- added R46: R001 DNI, Resistors_SMD:R_2512, B.Cu at (26.6, 35.0)
- added R47: 120R, Resistors_SMD:R_0603_HandSoldering, F.Cu at (25.9, 34.0)
- added R48: 120R, Resistors_SMD:R_0603_HandSoldering, F.Cu at (25.9, 35.5)
- added R49: 1k, Resistors_SMD:R_0603_HandSoldering, F.Cu at (35.0, 35.9)
- added R50: 120R, Resistors_SMD:R_0603_HandSoldering, F.Cu at (34.0, 32.5)
- added R51: 0.01R, Resistors_SMD:R_2512, F.Cu at (112.6, 92.4)
- added R52: R001 DNI, Resistors_SMD:R_2512, F.Cu at (112.6, 96.3)
- added R53: 120R, Resistors_SMD:R_0603_HandSoldering, B.Cu at (114.5, 92.8)
- added R54: 120R, Resistors_SMD:R_0603_HandSoldering, B.Cu at (114.5, 95.5)
- added R55: 1k, Resistors_SMD:R_0603_HandSoldering, B.Cu at (103.8, 95.5)
- added R56: 120R, Resistors_SMD:R_0603_HandSoldering, B.Cu at (106.0, 92.8)
- added U7: LT6105, components:MSOP-8_3x3mm_Pitch0.65mm-thin, F.Cu at (30.5, 35.0)
- added U8: LT6105, components:MSOP-8_3x3mm_Pitch0.65mm-thin, B.Cu at (110.2, 94.5)
- R33: value 120R -> 0.01R; footprint Resistors_SMD:R_0603_HandSoldering -> Resistors_SMD:R_2512; moved to B.Cu
- R34, R40: value 120R -> R001 DNI; footprint Resistors_SMD:R_0603_HandSoldering -> Resistors_SMD:R_2512; moved to B.Cu
- R35: value 1k -> 120R
- R36: value 0.01R -> 120R; footprint Resistors_SMD:R_2512 -> Resistors_SMD:R_0603_HandSoldering; moved to F.Cu
- R37: value 0.01R -> 1k; footprint Resistors_SMD:R_2512 -> Resistors_SMD:R_0603_HandSoldering; moved to F.Cu
- R38: value R001 DNI -> 120R; footprint Resistors_SMD:R_2512 -> Resistors_SMD:R_0603_HandSoldering; moved to F.Cu
- R39: value R001 DNI -> 0.01R
- U5, U6: footprint Housings_SSOP:MSOP-8_3x3mm_Pitch0.65mm -> components:MSOP-8_3x3mm_Pitch0.65mm-thin
- moved R36 57.5 mm to (54.4, 34.0), turned to 0 degrees
- moved R42 49.2 mm to (106.5, 35.7)
- moved R43 13.2 mm to (115.0, 35.5), turned to 270 degrees
- moved R44 11.6 mm to (114.0, 32.5), turned to 180 degrees
- moved C20 9.36 mm to (113.1, 35.2), turned to 270 degrees
- moved R38 6.76 mm to (56.9, 38.3), turned to 0 degrees
- moved R41 5.92 mm to (106.5, 34.2), turned to 0 degrees
- moved R37 5.41 mm to (55.8, 36.0), turned to 0 degrees
- moved J8 4.60 mm to (116.0, 108.1)
- moved R35 4.57 mm to (54.4, 32.4), turned to 0 degrees
- moved U6 3.54 mm to (110.5, 33.5), turned to 90 degrees
- moved D9 2.75 mm to (63.2, 39.0), turned to 180 degrees
- moved R33 2.33 mm to (57.9, 32.4), turned to 90 degrees
- moved R34 2.19 mm to (54.1, 32.4), turned to 90 degrees
- moved R39 1.96 mm to (107.0, 35.2), turned to 270 degrees
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Connections:
- C19 pad 1: /IOUT_P -> /VOUT
- D3 pad 1: /IOUT_N -> /VOUT2
- D5 pad 2: /VS -> /VS2
- J5 pad 2: /IOUT_N -> /VOUT2
- J6 pad 2: /IOUT_N -> /VOUT2
- J8 pad 2: /VBUS_COM -> /VBUS_COM_IN
- Q11 pad 2: /IOUT_P -> /VOUT
- Q12 pad 2: /VS -> /VS2
- Q14 pad 2: /IOUT_P -> /VOUT
- Q3 pad 2: /VS -> /VS2
- Q6 pad 2: /ICHARGE_N -> /CCCV_IN2
- R33 pad 1: /CCCV_IN -> /CCCV_IN2
- R33 pad 2: Net-(R33-Pad2) -> /CCCV_IN
- R34 pad 1: /ICHARGE_N -> /CCCV_IN2
- R34 pad 2: Net-(R34-Pad2) -> /CCCV_IN
- R35 pad 1: Net-(R35-Pad1) -> /CCCV_IN
- R35 pad 2: GND -> Net-(R35-Pad2)
- R36 pad 1: /IOUT_P -> /CCCV_IN2
- R36 pad 2: /IOUT_N -> Net-(R36-Pad2)
- R37 pad 1: /CCCV_IN -> Net-(R37-Pad1)
- R37 pad 2: /ICHARGE_N -> GND
- R38 pad 1: /CCCV_IN -> Net-(R37-Pad1)
- R38 pad 2: /ICHARGE_N -> /ICHARGE_SENS
- R39 pad 1: /IOUT_P -> /VOUT2
- R39 pad 2: /IOUT_N -> /VOUT
- R40 pad 1: /IOUT_P -> /VOUT2
- R40 pad 2: Net-(R40-Pad2) -> /VOUT
- R41 pad 1: /IOUT_N -> /VOUT
- R42 pad 1: Net-(R35-Pad1) -> /VOUT2
- R42 pad 2: /ICHARGE_SENS -> Net-(R42-Pad2)
- U1 pad 27: /GPIO_AUX2 -> /ISYS_SENS
- U1 pad 28: /GPIO_AUX3 -> /IUSB_SENS
- U1 pad 5: Net-(U1-Pad5) -> /GPIO_AUX2
- U1 pad 6: Net-(U1-Pad6) -> /GPIO_AUX3
- U5 pad 1: Net-(R34-Pad2) -> Net-(R36-Pad2)
- U5 pad 8: Net-(R33-Pad2) -> Net-(R35-Pad2)
- U6 pad 1: Net-(R41-Pad2) -> Net-(R42-Pad2)
- U6 pad 8: Net-(R40-Pad2) -> Net-(R41-Pad2)
Routing:
- net GND: track 252.0 -> 398.7 mm, vias 130 -> 151
- net +5V: track 216.0 -> 295.0 mm, vias 0 -> 4
- net /IUSB_SENS: track 0.00 -> 75.4 mm, vias 0 -> 1
- net /ISYS_SENS: track 0.00 -> 68.4 mm, vias 0 -> 2
- net /VS2: track 0.00 -> 18.8 mm, vias 0 -> 1
- net /GPIO_AUX3: track 4.87 -> 20.7 mm
- net /VOUT: track 0.00 -> 11.5 mm
- net /VOUT2: track 0.00 -> 9.34 mm, vias 0 -> 1
- net /GPIO_AUX2: track 4.87 -> 13.7 mm
- net /IOUT_SENS: track 107.0 -> 115.8 mm
- net Net-(R35-Pad2): track 0.00 -> 8.40 mm
- net Net-(R33-Pad2): track 7.15 -> 0.00 mm
- net /CCCV_IN2: track 0.00 -> 7.13 mm, vias 0 -> 1
- net /SW_VR1: track 63.4 -> 69.9 mm
- net /VBUS_COM_IN: track 0.00 -> 5.97 mm, vias 0 -> 1
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- added copper zone on B.Cu, net /CCCV_IN2
- added copper zone on F.Cu, net /VBUS_COM
- added copper zone on F.Cu, net /VBUS_COM_IN
- added copper zone on B.Cu, net /VOUT
- added copper zone on B.Cu, net /VOUT2
- added copper zone on B.Cu, net /VS2
- removed copper zone on B.Cu, net /ICHARGE_N
- removed copper zone on B.Cu, net /IOUT_N
- removed copper zone on B.Cu, net /IOUT_P
Other:
- board text added: "+ -"

Commit message: Some architectual changes
Parts:
- added C24: 0.1u, Capacitors_ThroughHole:C_Disc_D4.3mm_W1.9mm_P5.00mm, F.Cu at (172.8, 73.8)
- added C25: 1u, Capacitors_SMD:C_0603_HandSoldering, F.Cu at (171.3, 104.3)
- added C69: 10u, Capacitors_SMD:C_1206_HandSoldering, F.Cu at (248.5, 27.0)
- added D26: ESD5Z3.3T1G, Diodes_SMD:D_SOD-523, F.Cu at (173.5, 115.4)
- added D27: ESD5Z3.3T1G, Diodes_SMD:D_SOD-523, F.Cu at (183.9, 98.5)
- added D28: ESD5Z3.3T1G, Diodes_SMD:D_SOD-523, F.Cu at (163.1, 115.4)
- added D29: ESD5Z3.3T1G, Diodes_SMD:D_SOD-523, F.Cu at (152.7, 115.4)
- added D30: 6V, Diodes_SMD:D_SMA_Handsoldering, F.Cu at (166.1, 72.0)
- added D31: ESD5Z3.3T1G, Diodes_SMD:D_SOD-523, F.Cu at (176.6, 64.0)
- added D32: ESD5Z3.3T1G, Diodes_SMD:D_SOD-523, F.Cu at (176.6, 59.3)
- added D33: ESD5Z3.3T1G, Diodes_SMD:D_SOD-523, F.Cu at (209.6, 59.3)
- added J18: Conn_01x03_Female, components:Push_Terminal_3P_2.54, F.Cu at (155.4, 96.4)
- added J19: USB_B_Micro, components:USB-MICRO-B-RECEPT-UNIVERSAL, F.Cu at (166.2, 65.5)
- added J20: Conn_01x10_Male, Pin_Headers:Pin_Header_Straight_1x10_Pitch2.54mm, F.Cu at (258.0, 49.9)
- added JP3: Jumper_NO_Small, components:SolderJumper, F.Cu at (154.4, 110.1)
- added JP6: Jumper_NC_Small, components:SolderJumper, F.Cu at (171.8, 99.1)
- added Q18: Q_PNP_BEC, TO_SOT_Packages_SMD:SOT-23_Handsoldering, F.Cu at (200.9, -1.12)
- added R57: 22k, Resistors_SMD:R_0603_HandSoldering, F.Cu at (204.9, 0.38)
- added R58: 10k, Resistors_SMD:R_0603_HandSoldering, F.Cu at (202.0, 1.38)
- added R59: 10k, Resistors_SMD:R_0603_HandSoldering, F.Cu at (198.4, 1.88)
- added R60: 1k, Resistors_SMD:R_0603_HandSoldering, F.Cu at (201.5, -3.62)
- added R61: 22k, Resistors_SMD:R_0603_HandSoldering, F.Cu at (167.1, 104.5)
- added R62: 22k, Resistors_SMD:R_0603_HandSoldering, F.Cu at (163.5, 78.1)
- added R63: 22k, Resistors_SMD:R_0603_HandSoldering, F.Cu at (173.6, 68.9)
- added R64: 680, Resistors_SMD:R_0603_HandSoldering, F.Cu at (177.9, 68.9)
- added R65: 10k, Resistors_SMD:R_0603_HandSoldering, F.Cu at (184.0, 59.4)
- added R66: 0R, Resistors_SMD:R_0603_HandSoldering, F.Cu at (222.0, 100.5)
- added U10: P82B715, Housings_SOIC:SOIC-8_3.9x4.9mm_Pitch1.27mm, F.Cu at (192.8, 105.4)
- added U9: LM393, Housings_SOIC:SO-8_5.3x6.2mm_Pitch1.27mm, F.Cu at (203.3, 8.19)
- C4: value 1u -> 4.7u; footprint Capacitors_SMD:C_0603_HandSoldering -> Capacitors_SMD:C_0805_HandSoldering
- C5, C7: value 100u -> 1u; footprint Capacitors_ThroughHole:CP_Radial_D8.0mm_P2.50mm -> Capacitors_SMD:C_0603_HandSoldering
- D15, D16, D17, D18, D19, D20, D21, D22: footprint Diodes_SMD:D_SMA_Handsoldering -> Diodes_SMD:D_SMA; moved to B.Cu
- F1, F10, F11, F12, F13, F14, F15, F16, F2, F3, F4, F5, F6, F7, F8, F9: footprint Fuse_Holders_and_Fuses:Fuse_SMD1206_HandSoldering -> Fuse_Holders_and_Fuses:Fuse_SMD1206_Wave
- J14: value Conn_01x05_Female -> Conn_01x04_Male; footprint Pin_Headers:Pin_Header_Straight_1x05_Pitch2.54mm -> Pin_Headers:Pin_Header_Straight_1x04_Pitch2.54mm
- Q16: value Q_NPN_BEC -> Q_Photo_NPN_EC; footprint TO_SOT_Packages_SMD:SOT-23_Handsoldering -> LEDs:LED_D3.0mm
- Q17: value Q_PMOS_GSD -> Q_NPN_BEC
- R20, R23: value 10k -> 22k
- R31: value 10k -> 4.7k
- R32: value 470k -> 4.7k
- R34, R40: value R001 DNI -> 2.2k; footprint Resistors_SMD:R_2512 -> Resistors_SMD:R_0603_HandSoldering
- R46: value R001 DNI -> 100k; footprint Resistors_SMD:R_2512 -> Resistors_SMD:R_0603_HandSoldering; moved to F.Cu
- R52: value R001 DNI -> 100k; footprint Resistors_SMD:R_2512 -> Resistors_SMD:R_0603_HandSoldering
- U1: value ATMEGA328P-PU -> ATMEGA328P-AU; footprint Housings_DIP:DIP-28_W7.62mm_Socket -> Housings_QFP:TQFP-32_7x7mm_Pitch0.8mm
- U2: value L7805 -> L7803
- U3: value ATTINY2313-20PU -> ATTINY2313-20SU; footprint Housings_DIP:DIP-20_W7.62mm -> Housings_SOIC:SOIC-20W_7.5x12.8mm_Pitch1.27mm
- U4: value ATTINY13A-PU -> ATTINY13A-SSU; footprint Housings_DIP:DIP-8_W7.62mm -> Housings_SOIC:SOIC-8_3.9x4.9mm_Pitch1.27mm
- moved R34 255.4 mm to (309.5, 27.5)
- moved R40 199.1 mm to (307.0, 1.60)
- moved U1 188.2 mm to (232.5, 53.5)
- moved C19 182.8 mm to (286.4, -1.20)
- moved C20 182.8 mm to (290.1, -10.3)
- moved BT1 182.8 mm to (200.1, 46.1)
- moved C1 182.8 mm to (240.6, 35.9)
- moved C10 182.8 mm to (269.8, 37.4)
- moved C17 182.8 mm to (202.5, 25.6)
- moved C18 182.8 mm to (207.9, 32.8)
- moved C2 182.8 mm to (240.7, 37.8)
- moved C21 182.8 mm to (237.0, -9.50)
- moved C22 182.8 mm to (210.0, -6.95)
- moved C3 182.8 mm to (240.6, 34.4)
- moved C4 182.8 mm to (242.1, 26.5)
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Connections:
- C1 pad 1: +5V -> +3V3
- C10 pad 1: +5V -> VCOM
- C2 pad 1: +5V -> +3V3
- C20 pad 1: +5V -> +3V3
- C21 pad 1: +5V -> +3V3
- C22 pad 1: +5V -> +3V3
- C23 pad 1: +5V -> +3V3
- C5 pad 1: Net-(C4-Pad1) -> Net-(C5-Pad1)
- C6 pad 1: +5V -> Net-(C6-Pad1)
- C7 pad 1: +5V -> /CCCV_OUT
- F1 pad 2: /VBUS_COM -> VCOM
- F10 pad 2: /VBUS_COM -> VCOM
- F11 pad 2: /VBUS_COM -> VCOM
- F12 pad 2: /VBUS_COM -> VCOM
- F13 pad 2: /VBUS_COM -> VCOM
- F14 pad 2: /VBUS_COM -> VCOM
- F15 pad 2: /VBUS_COM -> VCOM
- F16 pad 2: /VBUS_COM -> VCOM
- F2 pad 2: /VBUS_COM -> VCOM
- F3 pad 2: /VBUS_COM -> VCOM
- F4 pad 2: /VBUS_COM -> VCOM
- F5 pad 2: /VBUS_COM -> VCOM
- F6 pad 2: /VBUS_COM -> VCOM
- F7 pad 2: /VBUS_COM -> VCOM
- F8 pad 2: /VBUS_COM -> VCOM
- F9 pad 2: /VBUS_COM -> VCOM
- J10 pad 2: +5V -> VCOM
- J10 pad 3: /WaterLevel/SCK -> SCL
- J10 pad 4: /WaterLevel/MOSI -> SDA
- J14 pad 2: /GPIO_AUX1 -> +3V3
- J14 pad 3: /GPIO_AUX2 -> Net-(D27-Pad1)
- J14 pad 4: /GPIO_AUX3 -> Net-(D28-Pad1)
- J15 pad 4: +5V -> VCOM
- J3 pad 1: GND -> /CCCV_FEEDBACK
- J7 pad 2: +5V -> +3V3
- Q16 pad 1: Net-(Q16-Pad1) -> /WaterLevel/SENS
- Q16 pad 2: GND -> /WaterLevel/CHARGE
- Q17 pad 1: Net-(Q16-Pad3) -> Net-(Q17-Pad1)
- Q17 pad 2: /VA_G -> GND
- Q17 pad 3: Net-(Q17-Pad3) -> Net-(J20-Pad2)
- R23 pad 1: Net-(Q17-Pad3) -> /VA_G
- R3 pad 1: +5V -> +3V3
- R30 pad 1: /WaterLevel/MOSI -> SDA
- R31 pad 1: /VA_SENS_EN -> +3V3
- R31 pad 2: Net-(Q16-Pad1) -> SCL
- R32 pad 1: /VA_G -> +3V3
- R32 pad 2: Net-(Q16-Pad3) -> SDA
- R34 pad 1: /CCCV_IN2 -> +3V3
- R34 pad 2: /CCCV_IN -> Net-(D28-Pad1)
- R40 pad 1: /VOUT2 -> +3V3
- R40 pad 2: /VOUT -> Net-(D27-Pad1)
- R46 pad 1: /VS2 -> /CC_CTRL
- R46 pad 2: /VS -> Net-(C5-Pad1)
- R51 pad 1: /VBUS_COM -> VCOM
- R52 pad 1: /VBUS_COM -> /CV_CTRL
- R52 pad 2: /VBUS_COM_IN -> Net-(C6-Pad1)
- R54 pad 1: /VBUS_COM -> VCOM
- U1 pad 1: /~RESET -> Net-(U1-Pad1)
- U1 pad 10: Net-(U1-Pad10) -> /SW_VR2
- U1 pad 11: /SW_VR1 -> /SW_BAT
- U1 pad 12: /SW_VR2 -> /SW_VS
- U1 pad 13: /SW_BAT -> /CC_CTRL
- U1 pad 14: /SW_VS -> /CV_CTRL
- U1 pad 15: /~DEEP_SLEEP_EN -> /MOSI
- U1 pad 16: /VA_SENS_EN -> /MISO
- U1 pad 17: /MOSI -> /SCK
- U1 pad 18: /MISO -> +3V3
- U1 pad 19: /SCK -> /BAT_TEMP_SENS
- U1 pad 2: /RX -> Net-(U1-Pad2)
- U1 pad 20: +5V -> Net-(C3-Pad1)
- U1 pad 21: Net-(C3-Pad1) -> Net-(U1-Pad21)
- U1 pad 22: GND -> /ICHARGE_SENS
- U1 pad 25: /ICHARGE_SENS -> /IOUT_SENS
- U1 pad 26: /IOUT_SENS -> /ISYS_SENS
- U1 pad 27: /ISYS_SENS -> SDA
- U1 pad 28: /IUSB_SENS -> SCL
- U1 pad 3: /TX -> GND
- U1 pad 4: /GPIO_AUX1 -> +3V3
- U1 pad 5: /GPIO_AUX2 -> GND
- U1 pad 6: /GPIO_AUX3 -> Net-(U1-Pad6)
- U1 pad 7: +5V -> /~DEEP_SLEEP_EN
- U1 pad 8: GND -> Net-(R61-Pad1)
- U1 pad 9: Net-(U1-Pad9) -> /SW_VR1
- U2 pad 3: +5V -> +3V3
- U3 pad 11: Net-(U3-Pad11) -> /WaterLevel/LCD_D7
- U3 pad 12: Net-(SW2-Pad2) -> /WaterLevel/SENS
- U3 pad 14: /WaterLevel/SENS -> Net-(SW2-Pad2)
- U3 pad 16: Net-(U3-Pad16) -> /WaterLevel/LED_LCD_PWM
- U3 pad 17: /WaterLevel/MOSI -> SDA
- U3 pad 19: /WaterLevel/SCK -> SCL
- U3 pad 20: +5V -> VCOM
- U3 pad 3: Net-(U3-Pad3) -> /WaterLevel/LCD_E
- U3 pad 6: Net-(U3-Pad6) -> /WaterLevel/LCD_RS
- U3 pad 7: Net-(U3-Pad7) -> /WaterLevel/LCD_D4
- U3 pad 8: Net-(U3-Pad8) -> /WaterLevel/LCD_D5
- U3 pad 9: Net-(U3-Pad9) -> /WaterLevel/LCD_D6
- U5 pad 2: +5V -> +3V3
- U6 pad 2: +5V -> +3V3
- U7 pad 2: +5V -> +3V3
- U8 pad 2: +5V -> +3V3
Routing:
- net GND: track 398.7 -> 0.00 mm, vias 151 -> 0
- net +5V: track 295.0 -> 0.00 mm, vias 4 -> 0
- net /VBUS_COM: track 146.0 -> 0.00 mm, vias 1 -> 0
- net /IOUT_SENS: track 115.8 -> 0.00 mm, vias 2 -> 0
- net /IUSB_SENS: track 75.4 -> 0.00 mm, vias 1 -> 0
- net /ICHARGE_SENS: track 72.4 -> 0.00 mm, vias 4 -> 0
- net /SW_VR2: track 71.9 -> 0.00 mm, vias 3 -> 0
- net /SW_VR1: track 69.9 -> 0.00 mm
- net /ISYS_SENS: track 68.4 -> 0.00 mm, vias 2 -> 0
- net /VS: track 62.3 -> 0.00 mm, vias 2 -> 0
- net Net-(C4-Pad1): track 52.9 -> 0.00 mm
- net /SW_BAT: track 49.0 -> 0.00 mm, vias 1 -> 0
- net /SW_VS: track 47.3 -> 0.00 mm, vias 1 -> 0
- net /~DEEP_SLEEP_EN: track 42.4 -> 0.00 mm, vias 1 -> 0
- net /SingleButtonRemocon/VBAT3V3: track 41.5 -> 0.00 mm, vias 3 -> 0
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- removed copper zone on B.Cu, net /BiDiSwitch1/COM_SRC
- removed copper zone on B.Cu, net /BiDiSwitch2/COM_SRC
- removed copper zone on B.Cu, net /BiDiSwitch3/COM_SRC
- removed copper zone on B.Cu, net /BiDiSwitch4/COM_SRC
- removed copper zone on B.Cu, net /CCCV_IN
- removed copper zone on B.Cu, net /CCCV_IN2
- removed copper zone on B.Cu, net /CCCV_OUT
- removed copper zone on B.Cu, net /VA
- removed copper zone on F.Cu, net /VBUS_COM
- removed copper zone on F.Cu, net /VBUS_COM_IN
- removed copper zone on B.Cu, net /VOUT
- removed copper zone on B.Cu, net /VOUT2
- removed copper zone on B.Cu, net /VS
- removed copper zone on B.Cu, net /VS2
- removed copper zone on B.Cu, net GND
- removed copper zone on F.Cu, net GND
Other:
- board text added: "+ FB"

Commit message: Use voltage regulator's RUN(EN) control for enable/disable CCCV output
Parts:
- removed D10, D8: 12V, Diodes_SMD:D_1206
- removed D9: LED, LEDs:LED_D3.0mm
- removed Q3, Q5, Q6, Q8: AOD403, components:TO-263-2-with-holes
- removed Q4, Q7: Q_NPN_BEC, TO_SOT_Packages_SMD:SOT-23_Handsoldering
- removed R10, R6: 470k, Resistors_SMD:R_0603_HandSoldering
- removed R11, R7, R8: 10k, Resistors_SMD:R_0603_HandSoldering
- removed R5, R9: 2.2k, Resistors_SMD:R_0603_HandSoldering
- removed R62, R63: 22k, Resistors_SMD:R_0603_HandSoldering
- added J21: Conn_01x02, Terminal_Blocks:TerminalBlock_bornier-2_P5.08mm, F.Cu at (74.0, 24.0)
- added J22: Conn_01x03_Female, Pin_Headers:Pin_Header_Straight_1x03_Pitch2.54mm, F.Cu at (305.4, 57.5)
- C17, R27, U4: moved to B.Cu
- C18: moved to F.Cu
- C19: value 1600u 35V -> 1600u 50V
- D7: value LED -> ESD5Z3.3T1G; footprint LEDs:LED_D3.0mm -> Diodes_SMD:D_SOD-523
- R4: value 10k -> 1k
- moved D11 186.9 mm to (84.5, 66.5)
- moved D13 186.9 mm to (95.0, 66.5)
- moved D14 186.9 mm to (96.5, 56.5)
- moved Q12 186.9 mm to (89.4, 55.4)
- moved Q13 186.9 mm to (102.1, 52.1)
- moved Q14 186.9 mm to (101.4, 57.9)
- moved R16 186.9 mm to (102.0, 58.6)
- moved R17 186.9 mm to (100.0, 58.5)
- moved R18 186.9 mm to (93.1, 56.7)
- moved R19 186.9 mm to (97.3, 52.9)
- moved C19 183.1 mm to (110.0, 48.0)
- moved Q11 176.9 mm to (100.5, 39.0)
- moved U1 174.4 mm to (60.0, 79.5)
- moved U3 171.8 mm to (104.0, 93.0)
- moved J18 131.0 mm to (29.0, 62.0), turned to 270 degrees
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Connections:
- net /SW_VR1 renamed /SW_VR
- C19 pad 1: /VOUT -> /VOUT2
- D7 pad 1: GND -> /CHG_ONLY
- D7 pad 2: Net-(D7-Pad2) -> GND
- J2 pad 2: /CCCV_OUT -> /VS2
- J3 pad 1: /CCCV_FEEDBACK -> GND
- JP6 pad 1: Net-(JP6-Pad1) -> GND
- R23 pad 1: /VA_G -> /VA
- R33 pad 1: /CCCV_IN2 -> /VA
- R36 pad 1: /CCCV_IN2 -> /VA
- U1 pad 10: /SW_VR2 -> Net-(U1-Pad10)
- U1 pad 32: Net-(U1-Pad32) -> /CHG_ONLY
- U9 pad 8: /CCCV_OUT -> Net-(U9-Pad8)
Other:
- board text added: "RUN FB"
- board text added: "VR CNTRL"
- board text removed: "+ FB"

Commit message: Layout in advance
Parts:
- added D8: ESD5Z5.0T1G, Diodes_SMD:D_SOD-523, F.Cu at (113.0, 79.0)
- added J23: Conn_01x04_Male, Pin_Headers:Pin_Header_Straight_1x04_Pitch2.54mm, F.Cu at (109.5, 73.7)
- added J24: Conn_01x02, components:TerminalBlock_2_P_2.54mm, F.Cu at (24.0, 75.0)
- added REF***: M, components:MountingHole_3.2mm_M3, F.Cu at (116.0, 84.0)
- added REF***: M, components:MountingHole_3.2mm_M3, F.Cu at (24.0, 84.0)
- C23, D24, R53, R54, R55, R56, U8: moved to F.Cu
- D26: value ESD5Z3.3T1G -> ESD5Z5.0T1G; moved to B.Cu
- D27, D28, D29, D31, D32, D33, D7: value ESD5Z3.3T1G -> ESD5Z5.0T1G
- F1, F2, R4: moved to B.Cu
- J14: value Conn_01x04_Male -> Conn_01x02; footprint Pin_Headers:Pin_Header_Straight_1x04_Pitch2.54mm -> components:TerminalBlock_2_P_2.54mm
- J18: value Conn_01x03_Female -> Conn_01x02; footprint components:Push_Terminal_3P_2.54 -> components:TerminalBlock_2_P_2.54mm
- J21: footprint Terminal_Blocks:TerminalBlock_bornier-2_P5.08mm -> components:TerminalBlock_2_P_2.54mm
- J22: value Conn_01x03_Female -> Conn_01x02; footprint Pin_Headers:Pin_Header_Straight_1x03_Pitch2.54mm -> components:TerminalBlock_2_P_2.54mm
- moved R40 289.4 mm to (30.5, 87.0)
- moved R34 287.7 mm to (28.8, 90.5)
- moved J22 284.0 mm to (24.0, 96.0), turned to 270 degrees
- moved C18 236.1 mm to (26.0, 50.0), turned to 0 degrees
- moved C17 235.8 mm to (22.0, 44.0), turned to 270 degrees
- moved R26 234.3 mm to (22.0, 44.0)
- moved D23 233.9 mm to (24.5, 40.5), turned to 0 degrees
- moved U4 233.5 mm to (26.2, 51.2)
- moved R27 233.5 mm to (26.5, 46.2)
- moved Q15 233.2 mm to (26.5, 45.5)
- moved BT1 229.5 mm to (21.4, 63.4)
- moved J16 229.5 mm to (21.8, 47.8)
- moved SW1 229.5 mm to (26.2, 60.2)
- moved D24 228.0 mm to (26.5, 52.0), turned to 0 degrees
- moved R31 224.8 mm to (40.5, 95.5)
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Connections:
- net Net-(SW3-Pad2) renamed /WaterLevel/ALLOW_DISCHG
- C1 pad 1: +3V3 -> +5V
- C2 pad 1: +3V3 -> +5V
- C20 pad 1: +3V3 -> +5V
- C21 pad 1: +3V3 -> +5V
- C22 pad 1: +3V3 -> +5V
- C23 pad 1: +3V3 -> +5V
- C25 pad 1: +3V3 -> +5V
- C69 pad 1: +3V3 -> +5V
- C7 pad 1: /CCCV_OUT -> /VS2
- D27 pad 1: Net-(D27-Pad1) -> /SDA_L
- D28 pad 1: Net-(D28-Pad1) -> /SCL_L
- D33 pad 1: +3V3 -> +5V
- D7 pad 1: /CHG_ONLY -> /WaterLevel/PREFER_DISCHG
- J14 pad 2: +3V3 -> +5V
- J18 pad 2: +3V3 -> +5V
- J22 pad 1: GND -> /SDA_L
- J22 pad 2: +3V3 -> /SCL_L
- J7 pad 2: +3V3 -> +5V
- JP3 pad 2: +3V3 -> +5V
- Q18 pad 2: +3V3 -> +5V
- R3 pad 1: +3V3 -> +5V
- R31 pad 1: +3V3 -> +5V
- R32 pad 1: +3V3 -> +5V
- R34 pad 1: +3V3 -> +5V
- R34 pad 2: Net-(D28-Pad1) -> /SCL_L
- R40 pad 1: +3V3 -> +5V
- R40 pad 2: Net-(D27-Pad1) -> /SDA_L
- R57 pad 2: +3V3 -> +5V
- SW2 pad 2: Net-(SW2-Pad2) -> /WaterLevel/PREFER_DISCHG
- U1 pad 18: +3V3 -> +5V
- U1 pad 32: /CHG_ONLY -> Net-(U1-Pad32)
- U1 pad 4: +3V3 -> +5V
- U10 pad 2: SDA -> /SDA_L
- U10 pad 3: Net-(D27-Pad1) -> SDA
- U10 pad 6: Net-(D28-Pad1) -> SCL
- U10 pad 7: SCL -> /SCL_L
- U10 pad 8: +3V3 -> +5V
- U2 pad 3: +3V3 -> +5V
- U3 pad 14: Net-(SW2-Pad2) -> /WaterLevel/PREFER_DISCHG
- U5 pad 2: +3V3 -> +5V
- U6 pad 2: +3V3 -> +5V
- U7 pad 2: +3V3 -> +5V
- U8 pad 2: +3V3 -> +5V
- U9 pad 8: Net-(U9-Pad8) -> /VS2
Routing:
- net +5V: track 0.00 -> 298.0 mm, vias 0 -> 3
- net /IOUT_SENS: track 0.00 -> 54.6 mm
- net /IUSB_SENS: track 0.00 -> 45.9 mm
- net GND: track 0.00 -> 44.8 mm, vias 0 -> 1
- net /CCCV_FEEDBACK: track 0.00 -> 44.4 mm, vias 0 -> 3
- net /SingleButtonRemocon/VBAT3V3: track 0.00 -> 37.7 mm, vias 0 -> 2
- net VCOM: track 0.00 -> 37.5 mm, vias 0 -> 5
- net /ICHARGE_SENS: track 0.00 -> 35.4 mm, vias 0 -> 2
- net /VS2: track 0.00 -> 29.6 mm, vias 0 -> 3
- net /VA: track 0.00 -> 28.1 mm, vias 0 -> 2
- net /VS: track 0.00 -> 26.2 mm, vias 0 -> 3
- net /VOUT2: track 0.00 -> 26.1 mm, vias 0 -> 1
- net /VA_SENSE_ADC: track 0.00 -> 25.8 mm, vias 0 -> 2
- net /SW_VR: track 0.00 -> 24.0 mm, vias 0 -> 3
- net /~DEEP_SLEEP_EN: track 0.00 -> 23.9 mm, vias 0 -> 2
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- added copper zone on B.Cu, net /BiDiSwitch3/COM_SRC
- added copper zone on B.Cu, net /BiDiSwitch4/COM_SRC
- added copper zone on B.Cu, net /CCCV_IN
- added copper zone on B.Cu, net /VA
- added copper zone on F.Cu, net /VBUS_COM_IN
- added copper zone on B.Cu, net /VOUT
- added copper zone on B.Cu, net /VOUT2
- added copper zone on B.Cu, net /VS
- added copper zone on B.Cu, net /VS2
- added copper zone on B.Cu, net GND
- added copper zone on F.Cu, net GND
- added copper zone on F.Cu, net VCOM
